File: hardware/fx2grok-tiny/fx2grok-tiny.kicad_pcb (KiCad board)
At the start: 2 copper layers, 13 x 13 mm, 28 parts, among them IC1 CY7C68013A-56, P1 CONN_01X05, P2 CONN_01X05, U1 MICRO-USB-B-SMD, U2 MIC5319, Y1 24MHz

Commit message: Set solder mask clearance to 2mil / 0.05mm.
Other:
- rule pad_to_mask_clearance: 0.09906 -> 0.0508
Changed lines of the file:
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@@
     (pad_size 1.89992 1.89992)
     (pad_drill 0)
-    (pad_to_mask_clearance 0.09906)
+    (pad_to_mask_clearance 0.0508)
     (aux_axis_origin 0 0)
     (visible_elements FFFFFF19)
